Commit message: 1st Working Windows Version

File: ar3_description/urdf/ar3.urdf (robot description, URDF)
Before this commit: robot ar3, 7 links, 6 joints
Links:
- added link gripper_base_link, mass 0.0837131933946375; collision mesh filename=package://ar3_description/meshes/gripper_base_link.STL; visual mesh filename=package://ar3_description/meshes/gripper_base_link.STL
- added link left_gripper, mass 0.00654748908133538; collision mesh filename=package://ar3_description/meshes/left_gripper.STL; visual mesh filename=package://ar3_description/meshes/left_gripper.STL
- added link right_Gripper, mass 0.00651398591885153; collision mesh filename=package://ar3_description/meshes/right_Gripper.STL; visual mesh filename=package://ar3_description/meshes/right_Gripper.STL
Joints:
- added joint joint_7: type fixed, parent link_6, child gripper_base_link, origin xyz=-0.000294 0 0.0162 rpy=-1.57 0 0, axis 0 0 1
- added joint leftGripper: type prismatic, parent gripper_base_link, child left_gripper, origin xyz=0 -0.035575 -0.015225 rpy=1.5708 0 0, axis 1 0 0, limit lower=0 upper=0 effort=0 velocity=0
- added joint rightGripper: type prismatic, parent gripper_base_link, child right_Gripper, origin xyz=0 -0.035575 0.009925 rpy=-1.5708 0 3.1416, axis 1 0 0, limit lower=0 upper=0 effort=0 velocity=0

File: ar3_description/urdf/ar3.urdf.xacro (robot description, xacro)
@@ -201,3 +201,43 @@
     <limit lower="-2.5848326" upper="2.5848326" effort="0" velocity="0"/>
   </joint>
+  <link
+    name="gripper_base_link">
+    <inertial>
+      <origin
+        xyz="0.000201676352247788 -0.000271374020595348 0.0205764880482399"
+        rpy="0 0 0" />
+      <mass
+        value="0.0837131933946375" />
+      <inertia
+        ixx="1.27397176956936E-05"
+        ixy="-1.92472475737929E-07"
+        ixz="-2.59961702797386E-07"
+        iyy="3.03147660705332E-05"
+        iyz="-4.38487554539977E-07"
+        izz="3.76673423663697E-05" />
+    </inertial>
+    <visual>
+      <origin
+        xyz="0 0 0"
+        rpy="0 0 0" />
+      <geometry>
+        <mesh
+          filename="package://ar3_description/meshes/gripper_base_link.STL" />
+      </geometry>
+      <material
+        name="">
+        <color
+          rgba="0.792156862745098 0.819607843137255 0.933333333333333 1" />
+      </material>
+    </visual>
+    <collision>
+      <origin
+        xyz="0 0 0"
+        rpy="0 0 0" />
+      <geometry>
+        <mesh
+          filename="//ar3_description/meshes/gripper_base_link.STL" />
+      </geometry>
+    </collision>
+  </link>
 </robot>
